Commit message: setup of get obeservations and load random objects

File: jaw_gripper/resources/tote/toteA_large.urdf (robot description, URDF)
Before this commit: robot toteA_large, 1 links, 0 joints
Links:
- link base_link: geometry collision mesh filename=ToteA.L.Proxy.obj scale=1.7 1.7 1.1; visual mesh filename=ToteA.L.obj scale=2.21 2.21 1.43

Commit message: refactored env and resources directory

File: jaw_gripper/resources/tote/toteA_large.urdf (robot description, URDF)
Before this commit: robot toteA_large, 1 links, 0 joints
Links:
- link base_link: geometry collision mesh filename=ToteA.L.Proxy.obj scale=1.7 1.7 1.1; visual mesh filename=ToteA.L.obj scale=2.21 2.21 .3
